File: to-order-march-2025/small-fix-cards-panelized.brd (EAGLE design)
At the start: 47 x 26.7 mm, 29 parts, among them IC1 DG412-JT, IC2 DG412-JT, IC3 DG412-JT, IC4 SN74LVC2T45, IC5 SN74LVC2T45, X1 ROUND-IC-PIN, X2 ROUND-IC-PIN, X3 ROUND-IC-PIN, X4 ROUND-IC-PIN, X5 ROUND-IC-PIN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

Commit message: Moved and changed order
Parts:
- T1, T2, T3, T4: value (none) -> 2n3904
Other:
- board text added: "DCO select"
- board text added: "Mode A"
- board text added: "Mode B"
- board text added: "Out A"
- board text added: "Out B"
- board text added: "WF"
- board text added: "Wave"
- board text added: "switch v1.0"
Changed lines of the file:
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@@
 <grid distance="6.25" unitdist="mil" unit="mil" style="lines" multiple="1" display="yes" altdistance="5" altunitdist="mil" altunit="mil"/>
 <layers>
-<layer number="1" name="Top" color="4" fill="1" visible="yes" active="yes"/>
+<layer number="1" name="Top" color="4" fill="1" visible="no" active="yes"/>
 <layer number="2" name="Route2" color="16" fill="1" visible="no" active="no"/>
 <layer number="15" name="Route15" color="23" fill="1" visible="no" active="no"/>
@@
 <layer number="19" name="Unrouted" color="6" fill="1" visible="yes" active="yes"/>
 <layer number="20" name="Dimension" color="24" fill="1" visible="yes" active="yes"/>
-<layer number="21" name="tPlace" color="7" fill="1" visible="yes" active="yes"/>
+<layer number="21" name="tPlace" color="7" fill="1" visible="no" active="yes"/>
 <layer number="22" name="bPlace" color="7" fill="1" visible="yes" active="yes"/>
-<layer number="23" name="tOrigins" color="15" fill="1" visible="yes" active="yes"/>
+<layer number="23" name="tOrigins" color="15" fill="1" visible="no" active="yes"/>
 <layer number="24" name="bOrigins" color="15" fill="1" visible="yes" active="yes"/>
-<layer number="25" name="tNames" color="7" fill="1" visible="yes" active="yes"/>
+<layer number="25" name="tNames" color="7" fill="1" visible="no" active="yes"/>
 <layer number="26" name="bNames" color="7" fill="1" visible="yes" active="yes"/>
 <layer number="27" name="tValues" color="7" fill="1" visible="no" active="yes"/>
@@
 <layer number="37" name="tTest" color="7" fill="1" visible="no" active="yes"/>
 <layer number="38" name="bTest" color="7" fill="1" visible="no" active="yes"/>
-<layer number="39" name="tKeepout" color="4" fill="11" visible="yes" active="yes"/>
+<layer number="39" name="tKeepout" color="4" fill="11" visible="no" active="yes"/>
 <layer number="40" name="bKeepout" color="1" fill="11" visible="yes" active="yes"/>
-<layer number="41" name="tRestrict" color="4" fill="10" visible="yes" active="yes"/>
+<layer number="41" name="tRestrict" color="4" fill="10" visible="no" active="yes"/>
 <layer number="42" name="bRestrict" color="1" fill="10" visible="yes" active="yes"/>
 <layer number="43" name="vRestrict" color="2" fill="10" visible="no" active="yes"/>
@@
 <layer number="49" name="Reference" color="7" fill="1" visible="no" active="yes"/>
 <layer number="50" name="dxf" color="7" fill="1" visible="no" active="no"/>
-<layer number="51" name="tDocu" color="7" fill="1" visible="yes" active="yes"/>
+<layer number="51" name="tDocu" color="7" fill="1" visible="no" active="yes"/>
 <layer number="52" name="bDocu" color="7" fill="1" visible="yes" active="yes"/>
 <layer number="53" name="tGND_GNDA" color="7" fill="9" visible="no" active="no"/>
@@
 <text x="15.5575" y="4.7625" size="0.8128" layer="26" font="vector" rot="MR0">2</text>
 <text x="16.51" y="6.985" size="0.8128" layer="25" font="vector">4VOB</text>
+<text x="42.70375" y="23.33625" size="0.8128" layer="25" font="vector">4VOB</text>
+<text x="45.085" y="21.59" size="0.8128" layer="26" font="vector" rot="SMR90" align="bottom-center">Out A</text>
+<text x="42.8625" y="19.05" size="0.8128" layer="26" font="vector" rot="MR90">WF</text>
+<text x="30.7975" y="24.13" size="0.8128" layer="26" font="vector" rot="MR270">Wave</text>
+<text x="30.1625" y="19.05" size="0.8128" layer="26" font="vector" rot="MR90">WF</text>
+<text x="31.4325" y="21.2725" size="0.8128" layer="26" font="vector">1</text>
+<text x="38.4175" y="24.13" size="0.8128" layer="26" font="vector" rot="MR270">GND</text>
+<text x="35.8775" y="24.13" size="0.8128" layer="26" font="vector" rot="MR270">V-</text>
+<text x="35.2425" y="19.05" size="0.8128" layer="26" font="vector" rot="MR90">V+</text>
+<text x="37.7825" y="19.05" size="0.8128" layer="26" font="vector" rot="MR90">V L</text>
+<text x="43.4975" y="24.13" size="0.8128" layer="26" font="vector" rot="MR270">Wave</text>
+<text x="29.21" y="23.495" size="0.8128" layer="26" font="vector" rot="MR0">1</text>
+<text x="27.46375" y="23.33625" size="0.8128" layer="25" font="vector">DCO select</text>
+<text x="40.005" y="21.59" size="0.8128" layer="26" font="vector" rot="MR90" align="bottom-center">Mode A</text>
+<text x="32.385" y="21.59" size="0.8128" layer="26" font="vector" rot="MR90" align="bottom-center">Mode B</text>
+<text x="27.305" y="21.59" size="0.8128" layer="26" font="vector" rot="MR90" align="bottom-center">Out B</text>
+<text x="27.46375" y="18.89125" size="0.8128" layer="25" font="vector">switch v1.0</text>
 </plain>
 <attributes>
@@
 <attribute name="VALUE" x="13.0175" y="20.955" size="1.27" layer="27" rot="R270"/>
 </element>
-<element name="T2" library="transistor" library_urn="urn:adsk.eagle:library:402" package="SOT23-BEC" package3d_urn="urn:adsk.eagle:package:28748/2" value="" x="17.145" y="21.2725" smashed="yes" rot="R180">
+<element name="T2" library="transistor" library_urn="urn:adsk.eagle:library:402" package="SOT23-BEC" package3d_urn="urn:adsk.eagle:package:28748/2" value="2n3904" x="17.145" y="21.2725" smashed="yes" rot="R180">
 <attribute name="POPULARITY" value="0" x="17.145" y="21.2725" size="0.8128" layer="27" font="vector" rot="R180" display="off"/>
 <attribute name="VALUE" x="19.05" y="24.4475" size="1.27" layer="27" rot="R180"/>
@@
 <attribute name="VALUE" x="13.0175" y="4.445" size="1.27" layer="27" rot="R270"/>
 </element>
-<element name="T1" library="transistor" library_urn="urn:adsk.eagle:library:402" package="SOT23-BEC" package3d_urn="urn:adsk.eagle:package:28748/2" value="" x="17.145" y="4.7625" smashed="yes" rot="R180">
+<element name="T1" library="transistor" library_urn="urn:adsk.eagle:library:402" package="SOT23-BEC" package3d_urn="urn:adsk.eagle:package:28748/2" value="2n3904" x="17.145" y="4.7625" smashed="yes" rot="R180">
 <attribute name="POPULARITY" value="0" x="17.145" y="4.7625" size="0.8128" layer="27" font="vector" rot="R180" display="off"/>
 <attribute name="VALUE" x="19.05" y="7.9375" size="1.27" layer="27" rot="R180"/>
@@
 <attribute name="VALUE" x="39.6875" y="21.2725" size="1.27" layer="27" rot="R270"/>
 </element>
-<element name="T3" library="transistor" library_urn="urn:adsk.eagle:library:402" package="SOT23-BEC" package3d_urn="urn:adsk.eagle:package:28748/2" value="" x="29.845" y="21.59" smashed="yes">
+<element name="T3" library="transistor" library_urn="urn:adsk.eagle:library:402" package="SOT23-BEC" package3d_urn="urn:adsk.eagle:package:28748/2" value="2n3904" x="29.845" y="21.59" smashed="yes">
 <attribute name="POPULARITY" value="0" x="29.845" y="1.27" size="1.778" layer="27" display="off"/>
 <attribute name="VALUE" x="27.94" y="18.415" size="1.27" layer="27"/>
 </element>
-<element name="T4" library="transistor" library_urn="urn:adsk.eagle:library:402" package="SOT23-BEC" package3d_urn="urn:adsk.eagle:package:28748/2" value="" x="43.815" y="21.59" smashed="yes" rot="R180">
+<element name="T4" library="transistor" library_urn="urn:adsk.eagle:library:402" package="SOT23-BEC" package3d_urn="urn:adsk.eagle:package:28748/2" value="2n3904" x="43.815" y="21.59" smashed="yes" rot="R180">
 <attribute name="POPULARITY" value="0" x="47.9425" y="47.625" size="1.778" layer="27" rot="R180" display="off"/>
 <attribute name="VALUE" x="45.72" y="24.765" size="1.27" layer="27" rot="R180"/>
 </element>
 <element name="IC3" library="joakim" package="TSSOP16J" value="DG412-JT" x="36.83" y="21.59" smashed="yes" rot="R90">
-<attribute name="NAME" x="39.43" y="18.6725" size="1.27" layer="25" rot="R180"/>
 <attribute name="VALUE" x="40.08" y="25.8225" size="1.27" layer="27" rot="R180"/>
 </element>
